File: SCH-PCB/PCB/minikeeb/minikeeb.kicad_sch (KiCad schematic)
At the start: 86 parts, among them J1 OLED, SW10 SW_PUSH-Lily58-cache, SW11 SW_PUSH-Lily58-cache, SW12 SW_PUSH-Lily58-cache, SW13 SW_PUSH-Lily58-cache, SW14 SW_PUSH-Lily58-cache, SW15 SW_PUSH-Lily58-cache, SW16 SW_PUSH-Lily58-cache, SW17 SW_PUSH-Lily58-cache, SW18 SW_PUSH-Lily58-cache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

Commit message: DOC: update readme
Connections:
- net 18: now reaches LED27.2 (DOUT), LED37.4 (DIN)
- net 18: now also LED38.4 (DIN), LED9.2 (DOUT)
- net 6: now reaches LED31.4 (DIN), LED34.2 (DOUT)
- net 6: now also LED13.4 (DIN), LED16.2 (DOUT)
- net 5: now reaches LED33.2 (DOUT), LED34.4 (DIN)
- net 5: now also LED15.2 (DOUT), LED16.4 (DIN)
- net 15: now reaches LED17.2 (DOUT), LED18.4 (DIN)
- net 15: now also LED35.2 (DOUT), LED36.4 (DIN)
- net 14: now reaches LED12.2 (DOUT), LED17.4 (DIN)
- net 14: now also LED30.2 (DOUT), LED35.4 (DIN)
- net 4: now reaches LED29.2 (DOUT), LED33.4 (DIN)
- net 4: now also LED11.2 (DOUT), LED15.4 (DIN)
- net 10: now reaches LED2.2 (DOUT), LED3.4 (DIN)
- net 10: now also LED20.2 (DOUT), LED21.4 (DIN)
- net 9: now reaches LED2.4 (DIN), LED6.2 (DOUT)
- net 9: now also LED20.4 (DIN), LED24.2 (DOUT)
- net 13: now reaches LED12.4 (DIN), LED8.2 (DOUT)
- net 13: now also LED26.2 (DOUT), LED30.4 (DIN)
- net 12: now reaches LED5.2 (DOUT), LED8.4 (DIN)
- net 12: now also LED23.2 (DOUT), LED26.4 (DIN)
- net 3: now reaches LED25.2 (DOUT), LED29.4 (DIN)
- net 3: now also LED11.4 (DIN), LED7.2 (DOUT)
- net 2: now reaches LED22.2 (DOUT), LED25.4 (DIN)
- net 2: now also LED4.2 (DOUT), LED7.4 (DIN)
- net 8: now reaches LED10.2 (DOUT), LED6.4 (DIN)
- net 8: now also LED24.4 (DIN), LED28.2 (DOUT)
- net 7: now reaches LED10.4 (DIN), LED13.2 (DOUT)
- net 7: now also LED28.4 (DIN), LED31.2 (DOUT)
- net 17: now reaches LED27.4 (DIN), LED32.2 (DOUT)
- net 17: now also LED14.2 (DOUT), LED9.4 (DIN)
- net 16: now reaches LED32.4 (DIN), LED36.2 (DOUT)
- net 16: now also LED14.4 (DIN), LED18.2 (DOUT)
- net 11: now reaches LED21.2 (DOUT), LED23.4 (DIN)
- net 11: now also LED3.2 (DOUT), LED5.4 (DIN)
- net 1: now reaches LED19.2 (DOUT), LED22.4 (DIN)
- net 1: now also LED1.2 (DOUT), LED4.4 (DIN)
