File: SCH-PCB/PCB/minikeeb/minikeeb.kicad_pcb (KiCad board)
At the start: 2 copper layers, 99.8 x 91 mm, 86 parts, among them J1 OLED, SW10 SW_PUSH-Lily58-cache, SW11 SW_PUSH-Lily58-cache, SW12 SW_PUSH-Lily58-cache, SW13 SW_PUSH-Lily58-cache, SW14 SW_PUSH-Lily58-cache, SW15 SW_PUSH-Lily58-cache, SW16 SW_PUSH-Lily58-cache, SW17 SW_PUSH-Lily58-cache, SW18 SW_PUSH-Lily58-cache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

Commit message: DOC: update readme
Connections:
- LED1 pad 2: Net-(LED1-DOUT) -> /1
- LED10 pad 2: Net-(LED10-DOUT) -> /8
- LED10 pad 4: Net-(LED10-DIN) -> /7
- LED11 pad 2: Net-(LED11-DOUT) -> /4
- LED11 pad 4: Net-(LED11-DIN) -> /3
- LED12 pad 2: Net-(LED12-DOUT) -> /14
- LED12 pad 4: Net-(LED12-DIN) -> /13
- LED13 pad 2: Net-(LED10-DIN) -> /7
- LED13 pad 4: Net-(LED13-DIN) -> /6
- LED14 pad 2: Net-(LED14-DOUT) -> /17
- LED14 pad 4: Net-(LED14-DIN) -> /16
- LED15 pad 2: Net-(LED15-DOUT) -> /5
- LED15 pad 4: Net-(LED11-DOUT) -> /4
- LED16 pad 2: Net-(LED13-DIN) -> /6
- LED16 pad 4: Net-(LED15-DOUT) -> /5
- LED17 pad 2: Net-(LED17-DOUT) -> /15
- LED17 pad 4: Net-(LED12-DOUT) -> /14
- LED18 pad 2: Net-(LED14-DIN) -> /16
- LED18 pad 4: Net-(LED17-DOUT) -> /15
- LED19 pad 2: Net-(LED19-DOUT) -> /1
- LED2 pad 2: Net-(LED2-DOUT) -> /10
- LED2 pad 4: Net-(LED2-DIN) -> /9
- LED20 pad 2: Net-(LED20-DOUT) -> /10
- LED20 pad 4: Net-(LED20-DIN) -> /9
- LED21 pad 2: Net-(LED21-DOUT) -> /11
- LED21 pad 4: Net-(LED20-DOUT) -> /10
- LED22 pad 2: Net-(LED22-DOUT) -> /2
- LED22 pad 4: Net-(LED19-DOUT) -> /1
- LED23 pad 2: Net-(LED23-DOUT) -> /12
- LED23 pad 4: Net-(LED21-DOUT) -> /11
- LED24 pad 2: Net-(LED20-DIN) -> /9
- LED24 pad 4: Net-(LED24-DIN) -> /8
- LED25 pad 2: Net-(LED25-DOUT) -> /3
- LED25 pad 4: Net-(LED22-DOUT) -> /2
- LED26 pad 2: Net-(LED26-DOUT) -> /13
- LED26 pad 4: Net-(LED23-DOUT) -> /12
- LED27 pad 2: Net-(LED27-DOUT) -> /18
- LED27 pad 4: Net-(LED27-DIN) -> /17
- LED28 pad 2: Net-(LED24-DIN) -> /8
- LED28 pad 4: Net-(LED28-DIN) -> /7
- LED29 pad 2: Net-(LED29-DOUT) -> /4
- LED29 pad 4: Net-(LED25-DOUT) -> /3
- LED3 pad 2: Net-(LED3-DOUT) -> /11
- LED3 pad 4: Net-(LED2-DOUT) -> /10
- LED30 pad 2: Net-(LED30-DOUT) -> /14
- LED30 pad 4: Net-(LED26-DOUT) -> /13
- LED31 pad 2: Net-(LED28-DIN) -> /7
- LED31 pad 4: Net-(LED31-DIN) -> /6
- LED32 pad 2: Net-(LED27-DIN) -> /17
- LED32 pad 4: Net-(LED32-DIN) -> /16
- LED33 pad 2: Net-(LED33-DOUT) -> /5
- LED33 pad 4: Net-(LED29-DOUT) -> /4
- LED34 pad 2: Net-(LED31-DIN) -> /6
- LED34 pad 4: Net-(LED33-DOUT) -> /5
- LED35 pad 2: Net-(LED35-DOUT) -> /15
- LED35 pad 4: Net-(LED30-DOUT) -> /14
- LED36 pad 2: Net-(LED32-DIN) -> /16
- LED36 pad 4: Net-(LED35-DOUT) -> /15
- LED37 pad 4: Net-(LED27-DOUT) -> /18
- LED38 pad 4: Net-(LED38-DIN) -> /18
- LED4 pad 2: Net-(LED4-DOUT) -> /2
- LED4 pad 4: Net-(LED1-DOUT) -> /1
- LED5 pad 2: Net-(LED5-DOUT) -> /12
- LED5 pad 4: Net-(LED3-DOUT) -> /11
- LED6 pad 2: Net-(LED2-DIN) -> /9
- LED6 pad 4: Net-(LED10-DOUT) -> /8
- LED7 pad 2: Net-(LED11-DIN) -> /3
- LED7 pad 4: Net-(LED4-DOUT) -> /2
- LED8 pad 2: Net-(LED12-DIN) -> /13
- LED8 pad 4: Net-(LED5-DOUT) -> /12
- LED9 pad 2: Net-(LED38-DIN) -> /18
- LED9 pad 4: Net-(LED14-DOUT) -> /17
Routing:
- net VCC: track 0.00 -> 494.8 mm, vias 0 -> 27
- net row0: track 61.8 -> 136.7 mm, vias 0 -> 2
- net col4: track 97.7 -> 172.0 mm, vias 4 -> 8
- net col3: track 77.2 -> 141.3 mm, vias 8 -> 10
- net row1: track 59.8 -> 120.3 mm, vias 0 -> 1
- net /15: track 0.00 -> 56.7 mm, vias 0 -> 2
- net col2: track 83.5 -> 132.3 mm
- net col1: track 40.4 -> 86.8 mm, vias 5 -> 7
- net row3: track 31.9 -> 71.8 mm, vias 0 -> 3
- net /18: track 0.00 -> 39.2 mm, vias 0 -> 2
- net /5: track 0.00 -> 38.6 mm, vias 0 -> 2
- net /10: track 0.00 -> 37.8 mm, vias 0 -> 2
- net /9: track 0.00 -> 27.5 mm, vias 0 -> 3
- net /17: track 0.00 -> 26.5 mm, vias 0 -> 2
- net /3: track 0.00 -> 26.0 mm, vias 0 -> 3
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
Commit message: FEAT: updaet PCB
Parts:
- added JP10: Jumper_NO_Small, sofle:Jumper, B.Cu at (108.3, 130.6)
- added JP11: Jumper_NO_Small, sofle:Jumper, F.Cu at (108.4, 128.5)
- added JP12: Jumper_NO_Small, sofle:Jumper, F.Cu at (108.3, 130.6)
- added JP9: Jumper_NO_Small, sofle:Jumper, B.Cu at (108.3, 128.5)
- U2: footprint Keebio-Parts:TRRS-PJ-320A-no-Fmask-makenova-reversible -> sofle:MJ-4PP-9
- moved U2 0.96 mm to (126.1, 129.3)
Connections:
- U2 pad 2: GND -> Net-(U2-TIP)
- U2 pad 3: DATA0 -> Net-(U2-RING1)
- U2 pad 4: +5V -> VCC
- U3 pad 13: ench_b -> txd0
- U3 pad 14: unconnected-(U3-13-Pad14) -> rxd0
- U3 pad 15: unconnected-(U3-14-Pad15) -> SDA
- U3 pad 16: unconnected-(U3-15-Pad16) -> SCL
- U3 pad 17: unconnected-(U3-26-Pad17) -> ench_b
- U3 pad 2: DATA0 -> unconnected-(U3-1-Pad2)
Routing:
- net VCC: track 494.8 -> 621.0 mm, vias 27 -> 34
- net rxd0: track 0.00 -> 81.7 mm, vias 0 -> 5
- net txd0: track 0.00 -> 75.7 mm, vias 0 -> 5
- net SCL: track 0.00 -> 24.8 mm, vias 0 -> 1
- net Net-(U2-RING1): track 0.00 -> 24.3 mm, vias 0 -> 1
- net SDA: track 0.00 -> 23.6 mm, vias 0 -> 1
- net Net-(U2-TIP): track 0.00 -> 22.8 mm, vias 0 -> 1
- net col4: track 172.0 -> 182.8 mm, vias 8 -> 10
- net ench_b: track 34.0 -> 37.1 mm
- net ench_a: track 30.9 -> 33.2 mm
- net GND: track 0.00 -> 1.42 mm, vias 69 -> 72

Commit message: FEAT: change microcontroller to promicro layout
Parts:
- removed U3: rp2040-zero, keeb_mcu:rp2040-zero-tht
- added SW1: SW_PUSH-Lily58-cache, sofle:TACT_SWITCH_TVBP06, F.Cu at (40.3, 139.9)
- added U1: ProMicro_2-Lily58-cache, sofle:ArduinoProMicro-ZigZag-DoubleSided, B.Cu at (45.7, 139.2)
- moved J1 0.97 mm to (63.8, 143.9)
Routing:
- net col2: track 132.3 -> 153.8 mm
- net VCC: track 621.0 -> 600.7 mm
- net row1: track 120.3 -> 140.4 mm, vias 1 -> 2
- net din: track 53.7 -> 73.7 mm, vias 1 -> 2
- net txd0: track 75.7 -> 91.6 mm
- net rxd0: track 81.7 -> 97.5 mm
- net row3: track 71.4 -> 58.5 mm, vias 3 -> 1
- net SDA: track 23.6 -> 36.1 mm, vias 1 -> 2
- net col4: track 182.8 -> 170.6 mm
- net row2: track 76.2 -> 87.9 mm, vias 0 -> 3
- net row0: track 136.7 -> 147.1 mm, vias 2 -> 1
- net col1: track 86.8 -> 96.0 mm, vias 7 -> 8
- net col0: track 98.5 -> 107.6 mm, vias 4 -> 5
- net reset: track 0.00 -> 7.29 mm
- net ench_b: track 37.1 -> 32.4 mm, vias 1 -> 2
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Other:
- outline, holes or cut-outs redrawn

Commit message: FEAT: add logo and name
Parts:
- added G***: LOGO, gundam:gundam, F.Cu at (76.2, 110.0)
- added G***: LOGO, gundam:gundam, B.Cu at (76.2, 110.0)
Other:
- board text added: "Positron Elektronik"
- board text added: "minikeeb V1.0"
