File: SCH-PCB/PCB/minikeeb/minikeeb.kicad_pcb (KiCad board)
At the start: 2 copper layers, 99.9 x 94.6 mm, 98 parts, among them J1 OLED, J2 Conn_01x02_Pin, J3 Conn_01x02_Pin, SW1 SW_PUSH-Lily58-cache, SW10 SW_PUSH-Lily58-cache, SW11 SW_PUSH-Lily58-cache, SW12 SW_PUSH-Lily58-cache, SW13 SW_PUSH-Lily58-cache, SW14 SW_PUSH-Lily58-cache, SW15 SW_PUSH-Lily58-cache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

Commit message: FEAT: update pcb
Parts:
- moved SW1 1.91 mm to (40.2, 139.8)
Routing:
- net reset: track 7.42 -> 9.31 mm
- net Net-(U1-RAW): track 10.5 -> 9.28 mm
Other:
- outline, holes or cut-outs redrawn
Changed lines of the file:
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@@
   )
   (footprint "sofle:TACT_SWITCH_TVBP06" (layer "F.Cu")
-    (at 40.3 141.76)
+    (at 40.25 139.85)
     (property "Sheetfile" "minikeeb.kicad_sch")
     (property "Sheetname" "")
@@
   (gr_circle (center 100.4 67.8) (end 101.41 67.86)
     (stroke (width 0.05) (type default)) (fill none) (layer "Edge.Cuts"))
-  (gr_line (start 30.1 136.61) (end 30.00612 74.091781)
+  (gr_line (start 30.135 135.7) (end 30.00612 74.091781)
     (stroke (width 0.2) (type solid)) (layer "Edge.Cuts"))
-  (gr_line (start 30.06 145.83) (end 30.07066 154.87934)
+  (gr_line (start 30.06 146.45) (end 30.07066 154.87934)
     (stroke (width 0.2) (type default)) (layer "Edge.Cuts"))
   (gr_circle (center 64.1 67.6) (end 65.11 67.66)
@@
   (gr_circle (center 108.15 153.64) (end 109.16 153.7)
     (stroke (width 0.05) (type default)) (fill none) (layer "Edge.Cuts"))
-  (gr_line (start 34.73 136.61) (end 34.73 145.83)
+  (gr_line (start 34.765 135.7) (end 34.73 146.45)
     (stroke (width 0.2) (type default)) (layer "Edge.Cuts"))
   (gr_line (start 126.086306 72.400921) (end 126.16741 134.663015)
@@
   (gr_circle (center 31.88 151.55) (end 32.89 151.61)
     (stroke (width 0.05) (type default)) (fill none) (layer "Edge.Cuts"))
-  (gr_line (start 30.1 136.61) (end 34.73 136.61)
+  (gr_line (start 30.135 135.7) (end 34.765 135.7)
     (stroke (width 0.2) (type default)) (layer "Edge.Cuts"))
   (gr_line (start 103.689999 156.359588) (end 31.57066 156.37934)
@@
   (gr_arc (start 126.325658 135.333595) (mid 126.20751 135.007514) (end 126.16741 134.663015)
     (stroke (width 0.2) (type solid)) (layer "Edge.Cuts"))
-  (gr_line (start 34.73 145.83) (end 30.06 145.83)
+  (gr_line (start 34.73 146.45) (end 30.06 146.45)
     (stroke (width 0.2) (type default)) (layer "Edge.Cuts"))
   (gr_arc (start 103.689999 156.359588) (mid 103.906076 156.381211) (end 104.113583 156.445223)
@@
   (via (at 32.95 129.3) (size 0.8) (drill 0.4) (layers "F.Cu" "B.Cu") (free) (net 1))
   (via (at 76.4 129) (size 0.8) (drill 0.4) (layers "F.Cu" "B.Cu") (free) (net 1))
-  (via (at 37.25 137.9) (size 0.8) (drill 0.4) (layers "F.Cu" "B.Cu") (free) (net 1))
+  (via (at 37.85 136.45) (size 0.8) (drill 0.4) (layers "F.Cu" "B.Cu") (free) (net 1))
   (via (at 69.85 105.75) (size 0.8) (drill 0.4) (layers "F.Cu" "B.Cu") (free) (net 1))
   (via (at 71.95 78.2) (size 0.8) (drill 0.4) (layers "F.Cu" "B.Cu") (free) (net 1))
@@
   (segment (start 106.932118 129.732118) (end 106.932118 128.54) (width 0.254) (layer "B.Cu") (net 62))
   (segment (start 107.79962 130.04962) (end 107.65 129.9) (width 0.254) (layer "B.Cu") (net 62))
-  (segment (start 37.05 141.76) (end 36.6 142.21) (width 0.4) (layer "B.Cu") (net 67))
-  (segment (start 36.6 142.21) (end 36.6 142.95) (width 0.4) (layer "B.Cu") (net 67))
+  (segment (start 36.6 140.25) (end 36.6 142.95) (width 0.4) (layer "B.Cu") (net 67))
   (segment (start 36.6 142.95) (end 36.76 143.11) (width 0.4) (layer "B.Cu") (net 67))
   (segment (start 36.76 143.11) (end 36.76 148.9286) (width 0.4) (layer "B.Cu") (net 67))
-  (segment (start 38.23 144.32) (end 36.78 144.32) (width 0.4) (layer "F.Cu") (net 68))
-  (segment (start 36.78 144.32) (end 36.65 144.45) (width 0.4) (layer "F.Cu") (net 68))
-  (segment (start 35.9 146.6) (end 31.95 146.6) (width 0.4) (layer "F.Cu") (net 68))
-  (segment (start 36.65 145.85) (end 35.9 146.6) (width 0.4) (layer "F.Cu") (net 68))
-  (segment (start 31.95 146.6) (end 31.68 146.87) (width 0.4) (layer "F.Cu") (net 68))
-  (segment (start 31.68 146.87) (end 31.68 148.9286) (width 0.4) (layer "F.Cu") (net 68))
+  (segment (start 37 139.85) (end 36.6 140.25) (width 0.4) (layer "B.Cu") (net 67))
   (segment (start 36.65 144.45) (end 36.65 145.85) (width 0.4) (layer "F.Cu") (net 68))
+  (segment (start 31.68 148.9286) (end 33.6086 147) (width 0.4) (layer "F.Cu") (net 68))
+  (segment (start 36.65 145.85) (end 35.5 147) (width 0.4) (layer "F.Cu") (net 68))
+  (segment (start 36.78 144.32) (end 36.65 144.45) (width 0.4) (layer "F.Cu") (net 68))
+  (segment (start 33.6086 147) (end 35.5 147) (width 0.4) (layer "F.Cu") (net 68))
+  (segment (start 38.23 144.32) (end 36.78 144.32) (width 0.4) (layer "F.Cu") (net 68))
   (segment (start 36.48 151.67) (end 36.15 152) (width 0.4) (layer "F.Cu") (net 70))
   (segment (start 43.84 151.67) (end 36.48 151.67) (width 0.4) (layer "F.Cu") (net 70))
